Commit message: Gazebo

File: description/robot_core.xacro (robot description, xacro)
@@ -40,4 +40,7 @@
         </xacro:inertial_box>
     </link>
+    <gazebo reference="chassic">
+            <material>Gazebo/White</material>
+    </gazebo>
     <!-- LEFT WHEEL LINK-->
     <joint name="left_wheel_joint" type="continuous">
@@ -63,4 +66,7 @@
         </xacro:inertial_cylinder>
     </link>
+    <gazebo reference="left_wheel">
+            <material>Gazebo/Blue</material>
+    </gazebo>
     <!-- RIGHT WHEEL LINK-->
     <joint name="right_wheel_joint" type="continuous">
@@ -86,4 +92,7 @@
         </xacro:inertial_cylinder>
     </link>
+        <gazebo reference="right_wheel">
+            <material>Gazebo/Blue</material>
+        </gazebo>
     <!--CASTER WHEEL LINK-->
     <joint name="caster_wheel_joint" type="fixed">
@@ -108,3 +117,6 @@
         </xacro:inertial_sphere>
     </link>
+        <gazebo reference="caster_wheel">
+            <material>Gazebo/Black</material>
+        </gazebo>
 </robot>

Commit message: Created core URDF

File: description/robot_core.xacro (robot description, xacro)
@@ -14,7 +14,7 @@
         <color rgba="0 0 0 1"/>
     </material>
-    <!--BASE LINK-->
+    <!-- BASE LINK -->
     <link name="base_link">
-    </link>
+    </link >
     <joint name="chassis_joint" type="fixed">
         <parent link="base_link"/>
@@ -43,5 +43,5 @@
             <material>Gazebo/White</material>
     </gazebo>
-    <!-- LEFT WHEEL LINK-->
+    <!-- LEFT WHEEL LINK -->
     <joint name="left_wheel_joint" type="continuous">
         <parent link="base_link"/>
@@ -55,5 +55,5 @@
                 <cylinder length="0.04" radius="0.05" />
             </geometry>
-            <material name="blue"/>
+            <material name="black"/>
         </visual>
         <collision>
@@ -67,7 +67,7 @@
     </link>
     <gazebo reference="left_wheel">
-            <material>Gazebo/Blue</material>
+            <material>Gazebo/Black</material>
     </gazebo>
-    <!-- RIGHT WHEEL LINK-->
+    <!-- RIGHT WHEEL LINK -->
     <joint name="right_wheel_joint" type="continuous">
         <parent link="base_link"/>
@@ -81,5 +81,5 @@
                 <cylinder length="0.04" radius="0.05" />
             </geometry>
-            <material name="blue"/>
+            <material name="black"/>
         </visual>
         <collision>
@@ -92,8 +92,8 @@
         </xacro:inertial_cylinder>
     </link>
-        <gazebo reference="right_wheel">
-            <material>Gazebo/Blue</material>
-        </gazebo>
-    <!--CASTER WHEEL LINK-->
+    <gazebo reference="right_wheel">
+        <material>Gazebo/Black</material>
+    </gazebo>
+    <!-- CASTER WHEEL LINK -->
     <joint name="caster_wheel_joint" type="fixed">
         <parent link="chassis"/>
@@ -117,6 +117,6 @@
         </xacro:inertial_sphere>
     </link>
-        <gazebo reference="caster_wheel">
-            <material>Gazebo/Black</material>
-        </gazebo>
+    <gazebo reference="caster_wheel">
+        <material>Gazebo/Black</material>
+    </gazebo>
 </robot>
