Commit message: Before setup ros2_control

File: description/gazebo_control.xacro (robot description, xacro)
@@ -3,5 +3,5 @@
     <gazebo>
         <plugin name="diff_drive" filename="libgazebo_ros_diff_drive.so">
-            <!--Wheel Information-->
+            <!-- Wheel Information  -->
             <left_joint>left_wheel_joint</left_joint>
             <right_joint>right_wheel_joint</right_joint>

File: description/robot.urdf.xacro (robot description, xacro)
@@ -2,3 +2,7 @@
 <robot xmlns:xacro="http://www.ros.org/wiki/xacro"  name="robot">
     <xacro:include filename="robot_core.xacro"/>
+    <xacro:include filename="gazebo_control.xacro"/>
+    <xacro:include filename="lidar.xacro"/>
+    <xacro:include filename="camera.xacro"/>
+    <!-- <xacro:include filename="depth_camera.xacro"/> -->
 </robot>

File: description/robot_core.xacro (robot description, xacro)
@@ -14,7 +14,10 @@
         <color rgba="0 0 0 1"/>
     </material>
+    <material name="red">
+        <color rgba="1 0 0 1"/>
+    </material>
     <!-- BASE LINK -->
-    <link name="base_link">
-    </link >
+    <link name="base_link"></link >
+    <!-- CHASSIS LINK -->
     <joint name="chassis_joint" type="fixed">
         <parent link="base_link"/>
@@ -43,5 +46,5 @@
             <material>Gazebo/White</material>
     </gazebo>
-    <!-- LEFT WHEEL LINK -->
+    <!-- LEFT_WHEEL LINK -->
     <joint name="left_wheel_joint" type="continuous">
         <parent link="base_link"/>
@@ -53,5 +56,5 @@
         <visual>
             <geometry>
-                <cylinder length="0.04" radius="0.05" />
+                <cylinder length="0.04" radius="0.05"/>
             </geometry>
             <material name="black"/>
@@ -59,5 +62,5 @@
         <collision>
             <geometry>
-                <cylinder length="0.04" radius="0.05" />
+                <cylinder length="0.04" radius="0.05"/>
             </geometry>
         </collision>
@@ -69,5 +72,5 @@
             <material>Gazebo/Black</material>
     </gazebo>
-    <!-- RIGHT WHEEL LINK -->
+    <!-- RIGHT_WHEEL LINK -->
     <joint name="right_wheel_joint" type="continuous">
         <parent link="base_link"/>
@@ -79,5 +82,5 @@
         <visual>
             <geometry>
-                <cylinder length="0.04" radius="0.05" />
+                <cylinder length="0.04" radius="0.05"/>
             </geometry>
             <material name="black"/>
@@ -85,5 +88,5 @@
         <collision>
             <geometry>
-                <cylinder length="0.04" radius="0.05" />
+                <cylinder length="0.04" radius="0.05"/>
             </geometry>
         </collision>
@@ -95,5 +98,5 @@
         <material>Gazebo/Black</material>
     </gazebo>
-    <!-- CASTER WHEEL LINK -->
+    <!-- CASTER_WHEEL LINK -->
     <joint name="caster_wheel_joint" type="fixed">
         <parent link="chassis"/>
@@ -119,4 +122,7 @@
     <gazebo reference="caster_wheel">
         <material>Gazebo/Black</material>
+        <!-- Specify frition coefficient -->
+        <mu1 value="0.001"/>
+        <mu2 value="0.001"/>
     </gazebo>
 </robot>
